File: KiCad/papa-project-board.kicad_pcb (KiCad board)
At the start: 2 copper layers, 120 x 59 mm, 62 parts, among them J1 GOOD, J10 I2C Aux, J11 +3.3V, J12 +5V, J13 VIN, J14 Servo 1, J15 GND, J16 Sensor 2, J17 OLED, J18 AuxIO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

Commit message: Dimmed the power LED
Parts:
- R5: value 330R -> 4.7k
Changed lines of the file:
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@@
 			)
 		)
-		(property "Value" "330R"
+		(property "Value" "4.7k"
 			(at 5.08 0 270)
 			(layer "B.SilkS")
